Commit message: Cleaned up urdf link names

File: urdf/Legs.urdf (robot description, URDF)
Before this commit: robot Legs, 13 links, 12 joints
Links:
- removed link Legs__Body
- removed link Legs__Bottom_Left_Leg
- removed link Legs__Bottom_Right_Leg
- removed link Legs__Left_Ankle
- removed link Legs__Left_Foot
- removed link Legs__Left_Hip
- removed link Legs__Left_Toe
- removed link Legs__Right_Ankle
- removed link Legs__Right_Foot
- removed link Legs__Right_Hip
- removed link Legs__Right_Toe
- removed link Legs__Top_Left_Leg
- removed link Legs__Top_Right_Leg
- added link Body, mass 3.53324885586669; visual mesh filename=meshes/Body.STL scale=1 1 1
- added link Bottom_Left_Leg, mass 0.559939379300119; visual mesh filename=meshes/Bottom_Left_Leg.STL scale=1 1 1
- added link Bottom_Right_Leg, mass 0.562143515434244; visual mesh filename=meshes/Bottom_Right_Leg.STL scale=1 1 1
- added link Left_Ankle, mass 0.117207342953091; visual mesh filename=meshes/Left_Ankle.STL scale=1 1 1
- added link Left_Foot, mass 0.350801135347807; collision mesh filename=meshes/Left_Foot_col.STL scale=1 1 1; visual mesh filename=meshes/Left_Foot.STL scale=1 1 1
- added link Left_Hip, mass 0.437298303222343; visual mesh filename=meshes/Left_Hip.STL scale=1 1 1
- added link Left_Toe, mass 0.137471306967525; collision mesh filename=meshes/Left_Toe_col.STL scale=1 1 1; visual mesh filename=meshes/Left_Toe.STL scale=1 1 1
- added link Right_Ankle, mass 0.113529394776609; visual mesh filename=meshes/Right_Ankle.STL scale=1 1 1
- added link Right_Foot, mass 0.335422480362735; collision mesh filename=meshes/Right_Foot_col.STL scale=1 1 1; visual mesh filename=meshes/Right_Foot.STL scale=1 1 1
- added link Right_Hip, mass 0.429542604129865; visual mesh filename=meshes/Right_Hip.STL scale=1 1 1
- added link Right_Toe, mass 0.139661985071308; collision mesh filename=meshes/Right_Toe_col.STL scale=1 1 1; visual mesh filename=meshes/Right_Toe.STL scale=1 1 1
- added link Top_Left_Leg, mass 0.498661420183801; visual mesh filename=meshes/Top_Left_Leg.STL scale=1 1 1
- added link Top_Right_Leg, mass 0.473894644129491; visual mesh filename=meshes/Top_Right_Leg.STL scale=1 1 1
Joints:
- removed joint Legs__Body-Left_Hip
- removed joint Legs__Body-Right_Hip
- removed joint Legs__Bottom_Left_Leg-Left_Ankle
- removed joint Legs__Bottom_Right_Leg-Right_Ankle
- removed joint Legs__Left_Ankle-Left_Foot
- removed joint Legs__Left_Foot-Left_Toe
- removed joint Legs__Left_Hip-Top_Left_Leg
- removed joint Legs__Right_Ankle-Right_Foot
- removed joint Legs__Right_Foot-Right_Toe
- removed joint Legs__Right_Hip-Top_Right_Leg
- removed joint Legs__Top_Left_Leg-Bottom_Left_Leg
- removed joint Legs__Top_Right_Leg-Bottom_Right_Leg
- added joint Body-Left_Hip: type fixed, parent Body, child Left_Hip, origin xyz=-0.00302 -0.05556  0.53887 rpy=1.56568  0       1.57079, axis 0       0.00511 -0.99998, limit lower=0.0 upper=0.0 effort=1.0 velocity=0.0
- added joint Body-Right_Hip: type fixed, parent Body, child Right_Hip, origin xyz=0.00313  0.05556  0.53887 rpy=-1.56565  0.00509 -3.13647, axis -0.99997  0.00511  0.00509, limit lower=0.0 upper=0.0 effort=1.0 velocity=0.0
- added joint Bottom_Left_Leg-Left_Ankle: type fixed, parent Bottom_Left_Leg, child Left_Ankle, origin xyz=-0.00049 -0.19818  0.09846 rpy=0  0  0, axis 1  0  0, limit lower=0.0 upper=0.0 effort=1.0 velocity=0.0
- added joint Bottom_Right_Leg-Right_Ankle: type fixed, parent Bottom_Right_Leg, child Right_Ankle, origin xyz=-1.20000000e-04  -1.24340000e-01   1.83060000e-01 rpy=0  0  0, axis 1  0  0, limit lower=0.0 upper=0.0 effort=1.0 velocity=0.0
- added joint Left_Ankle-Left_Foot: type fixed, parent Left_Ankle, child Left_Foot, origin xyz=-0.00077 -0.00465 -0.07126 rpy=0  0  0, axis 0       0.192   -0.98139, limit lower=0.0 upper=0.0 effort=1.0 velocity=0.0
- added joint Left_Foot-Left_Toe: type fixed, parent Left_Foot, child Left_Toe, origin xyz=0.00451 -0.0209  -0.07227 rpy=0  0  0, axis 0.99797  0.06244  0.01221, limit lower=0.0 upper=0.0 effort=1.0 velocity=0.0
- added joint Left_Hip-Top_Left_Leg: type fixed, parent Left_Hip, child Top_Left_Leg, origin xyz=-8.05900000e-02  -1.00000000e-05   3.02000000e-03 rpy=0  0  0, axis 1  0  0, limit lower=0.0 upper=0.0 effort=1.0 velocity=0.0
- added joint Right_Ankle-Right_Foot: type fixed, parent Right_Ankle, child Right_Foot, origin xyz=-0.00079 -0.03467 -0.06476 rpy=0  0  0, axis 0       0.23816  0.97122, limit lower=0.0 upper=0.0 effort=1.0 velocity=0.0
- added joint Right_Foot-Right_Toe: type fixed, parent Right_Foot, child Right_Toe, origin xyz=-0.0044  -0.04886 -0.05474 rpy=0  0  0, axis 0.97972 -0.19459  0.04771, limit lower=0.0 upper=0.0 effort=1.0 velocity=0.0
- added joint Right_Hip-Top_Right_Leg: type fixed, parent Right_Hip, child Top_Right_Leg, origin xyz=0.00274 -0.0004  -0.07526 rpy=0.78539  1.56355 -2.35618, axis 1  0  0, limit lower=0.0 upper=0.0 effort=1.0 velocity=0.0
- added joint Top_Left_Leg-Bottom_Left_Leg: type fixed, parent Top_Left_Leg, child Bottom_Left_Leg, origin xyz=0.00407 -0.16882 -0.12412 rpy=0  0  0, axis 1  0  0, limit lower=0.0 upper=0.0 effort=1.0 velocity=0.0
- added joint Top_Right_Leg-Bottom_Right_Leg: type fixed, parent Top_Right_Leg, child Bottom_Right_Leg, origin xyz=0.00346 -0.20909  0.01388 rpy=0  0  0, axis 1  0  0, limit lower=0.0 upper=0.0 effort=1.0 velocity=0.0

Commit message: update joint type from fixed to revolute

File: urdf/Legs.urdf (robot description, URDF)
Before this commit: robot Legs, 13 links, 12 joints
Joints:
- joint Body-Left_Hip: type fixed -> revolute
- joint Body-Right_Hip: type fixed -> revolute
- joint Bottom_Left_Leg-Left_Ankle: type fixed -> revolute
- joint Bottom_Right_Leg-Right_Ankle: type fixed -> revolute
- joint Left_Ankle-Left_Foot: type fixed -> revolute
- joint Left_Foot-Left_Toe: type fixed -> revolute
- joint Left_Hip-Top_Left_Leg: type fixed -> revolute
- joint Right_Ankle-Right_Foot: type fixed -> revolute
- joint Right_Foot-Right_Toe: type fixed -> revolute
- joint Right_Hip-Top_Right_Leg: type fixed -> revolute
- joint Top_Left_Leg-Bottom_Left_Leg: type fixed -> revolute
- joint Top_Right_Leg-Bottom_Right_Leg: type fixed -> revolute

Commit message: added large, fake joint limits

File: urdf/Legs.urdf (robot description, URDF)
Before this commit: robot Legs, 13 links, 12 joints
Joints:
- joint Body-Left_Hip: limit lower=0.0 upper=0.0 effort=1.0 velocity=0.0 -> lower=-3.1 upper=3.1 effort=1.0 velocity=0.0
- joint Body-Right_Hip: limit lower=0.0 upper=0.0 effort=1.0 velocity=0.0 -> lower=-3.1 upper=3.1 effort=1.0 velocity=0.0
- joint Bottom_Left_Leg-Left_Ankle: limit lower=0.0 upper=0.0 effort=1.0 velocity=0.0 -> lower=-3.1 upper=3.1 effort=1.0 velocity=0.0
- joint Bottom_Right_Leg-Right_Ankle: limit lower=0.0 upper=0.0 effort=1.0 velocity=0.0 -> lower=-3.1 upper=3.1 effort=1.0 velocity=0.0
- joint Left_Ankle-Left_Foot: limit lower=0.0 upper=0.0 effort=1.0 velocity=0.0 -> lower=-3.1 upper=3.1 effort=1.0 velocity=0.0
- joint Left_Foot-Left_Toe: limit lower=0.0 upper=0.0 effort=1.0 velocity=0.0 -> lower=-3.1 upper=3.1 effort=1.0 velocity=0.0
- joint Left_Hip-Top_Left_Leg: limit lower=0.0 upper=0.0 effort=1.0 velocity=0.0 -> lower=-3.1 upper=3.1 effort=1.0 velocity=0.0
- joint Right_Ankle-Right_Foot: limit lower=0.0 upper=0.0 effort=1.0 velocity=0.0 -> lower=-3.1 upper=3.1 effort=1.0 velocity=0.0
- joint Right_Foot-Right_Toe: limit lower=0.0 upper=0.0 effort=1.0 velocity=0.0 -> lower=-3.1 upper=3.1 effort=1.0 velocity=0.0
- joint Right_Hip-Top_Right_Leg: limit lower=0.0 upper=0.0 effort=1.0 velocity=0.0 -> lower=-3.1 upper=3.1 effort=1.0 velocity=0.0
- joint Top_Left_Leg-Bottom_Left_Leg: limit lower=0.0 upper=0.0 effort=1.0 velocity=0.0 -> lower=-3.1 upper=3.1 effort=1.0 velocity=0.0
- joint Top_Right_Leg-Bottom_Right_Leg: limit lower=0.0 upper=0.0 effort=1.0 velocity=0.0 -> lower=-3.1 upper=3.1 effort=1.0 velocity=0.0

Commit message: runcaminantedynamics works. need to fix the contact points arrangement but they're there! also need to change 1 drake file for it to run

File: urdf/Legs.urdf (robot description, URDF)
Before this commit: robot Legs, 13 links, 12 joints
Links:
- link Left_Foot: geometry collision mesh filename=meshes/Left_Foot_col.STL scale=1 1 1; collision sphere radius=0.0
- link Right_Foot: geometry collision mesh filename=meshes/Right_Foot_col.STL scale=1 1 1; collision sphere radius=0.0

Commit message: move toe collision points to toe links

File: urdf/Legs.urdf (robot description, URDF)
Before this commit: robot Legs, 13 links, 12 joints
Links:
- link Left_Foot: geometry collision mesh filename=meshes/Left_Foot_col.STL scale=1 1 1; collision sphere radius=0.0
- link Left_Toe: geometry collision mesh filename=meshes/Left_Toe_col.STL scale=1 1 1; collision sphere radius=0.0
- link Right_Foot: geometry collision mesh filename=meshes/Right_Foot_col.STL scale=1 1 1; collision sphere radius=0.0
- link Right_Toe: geometry collision mesh filename=meshes/Right_Toe_col.STL scale=1 1 1; collision sphere radius=0.0

Commit message: runCaminanteBalancing gets far enough to launch the drake visualizer and get a cpp exception... probably because the initial conditions and a lot of parameters are made up. also had to change a lot of link names becuase drake has hard-coded link names that it looks for. also added 'transmission' elements to the urdf for control inputs

File: urdf/Legs.urdf (robot description, URDF)
Before this commit: robot Legs, 13 links, 12 joints
Links:
- removed link Body
- removed link Left_Foot
- removed link Left_Toe
- removed link Right_Foot
- removed link Right_Toe
- added link l_foot, mass 0.350801135347807; collision mesh filename=meshes/Left_Foot_col.STL scale=1 1 1; collision sphere radius=0.0
- added link l_toe, mass 0.137471306967525; collision mesh filename=meshes/Left_Toe_col.STL scale=1 1 1; collision sphere radius=0.0
- added link pelvis, mass 3.53324885586669; visual mesh filename=meshes/Body.STL scale=1 1 1
- added link r_foot, mass 0.335422480362735; collision mesh filename=meshes/Right_Foot_col.STL scale=1 1 1; collision sphere radius=0.0
- added link r_toe, mass 0.139661985071308; collision mesh filename=meshes/Right_Toe_col.STL scale=1 1 1; collision sphere radius=0.0
Joints:
- removed joint Body-Left_Hip
- removed joint Body-Right_Hip
- removed joint Bottom_Left_Leg-Left_Ankle
- removed joint Bottom_Right_Leg-Right_Ankle
- removed joint Left_Ankle-Left_Foot
- removed joint Left_Foot-Left_Toe
- removed joint Left_Hip-Top_Left_Leg
- removed joint Right_Ankle-Right_Foot
- removed joint Right_Foot-Right_Toe
- removed joint Right_Hip-Top_Right_Leg
- removed joint Top_Left_Leg-Bottom_Left_Leg
- removed joint Top_Right_Leg-Bottom_Right_Leg
- added joint Body_to_Left_Hip: type revolute, parent pelvis, child Left_Hip, origin xyz=-0.00302 -0.05556  0.53887 rpy=1.56568  0       1.57079, axis 0       0.00511 -0.99998, limit lower=-3.1 upper=3.1 effort=1.0 velocity=0.0
- added joint Body_to_Right_Hip: type revolute, parent pelvis, child Right_Hip, origin xyz=0.00313  0.05556  0.53887 rpy=-1.56565  0.00509 -3.13647, axis -0.99997  0.00511  0.00509, limit lower=-3.1 upper=3.1 effort=1.0 velocity=0.0
- added joint Bottom_Left_Leg_to_Left_Ankle: type revolute, parent Bottom_Left_Leg, child Left_Ankle, origin xyz=-0.00049 -0.19818  0.09846 rpy=0  0  0, axis 1  0  0, limit lower=-3.1 upper=3.1 effort=1.0 velocity=0.0
- added joint Bottom_Right_Leg_to_Right_Ankle: type revolute, parent Bottom_Right_Leg, child Right_Ankle, origin xyz=-1.20000000e-04  -1.24340000e-01   1.83060000e-01 rpy=0  0  0, axis 1  0  0, limit lower=-3.1 upper=3.1 effort=1.0 velocity=0.0
- added joint Left_Ankle_to_Left_Foot: type revolute, parent Left_Ankle, child l_foot, origin xyz=-0.00077 -0.00465 -0.07126 rpy=0  0  0, axis 0       0.192   -0.98139, limit lower=-3.1 upper=3.1 effort=1.0 velocity=0.0
- added joint Left_Foot_to_Left_Toe: type revolute, parent l_foot, child l_toe, origin xyz=0.00451 -0.0209  -0.07227 rpy=0  0  0, axis 0.99797  0.06244  0.01221, limit lower=-3.1 upper=3.1 effort=1.0 velocity=0.0
- added joint Left_Hip_to_Top_Left_Leg: type revolute, parent Left_Hip, child Top_Left_Leg, origin xyz=-8.05900000e-02  -1.00000000e-05   3.02000000e-03 rpy=0  0  0, axis 1  0  0, limit lower=-3.1 upper=3.1 effort=1.0 velocity=0.0
- added joint Right_Ankle_to_Right_Foot: type revolute, parent Right_Ankle, child r_foot, origin xyz=-0.00079 -0.03467 -0.06476 rpy=0  0  0, axis 0       0.23816  0.97122, limit lower=-3.1 upper=3.1 effort=1.0 velocity=0.0
- added joint Right_Foot_to_Right_Toe: type revolute, parent r_foot, child r_toe, origin xyz=-0.0044  -0.04886 -0.05474 rpy=0  0  0, axis 0.97972 -0.19459  0.04771, limit lower=-3.1 upper=3.1 effort=1.0 velocity=0.0
- added joint Right_Hip_to_Top_Right_Leg: type revolute, parent Right_Hip, child Top_Right_Leg, origin xyz=0.00274 -0.0004  -0.07526 rpy=0.78539  1.56355 -2.35618, axis 1  0  0, limit lower=-3.1 upper=3.1 effort=1.0 velocity=0.0
- added joint Top_Left_Leg_to_Bottom_Left_Leg: type revolute, parent Top_Left_Leg, child Bottom_Left_Leg, origin xyz=0.00407 -0.16882 -0.12412 rpy=0  0  0, axis 1  0  0, limit lower=-3.1 upper=3.1 effort=1.0 velocity=0.0
- added joint Top_Right_Leg_to_Bottom_Right_Leg: type revolute, parent Top_Right_Leg, child Bottom_Right_Leg, origin xyz=0.00346 -0.20909  0.01388 rpy=0  0  0, axis 1  0  0, limit lower=-3.1 upper=3.1 effort=1.0 velocity=0.0

Commit message: fixed joint names

File: urdf/Legs.urdf (robot description, URDF)
Before this commit: robot Legs, 13 links, 12 joints
Joints:
- removed joint Biped__Body-Left_Hip
- removed joint Biped__Body-Right_Hip
- removed joint Biped__Bottom_Left_Leg-Left_Ankle
- removed joint Biped__Bottom_Right_Leg-Right_Ankle
- removed joint Biped__Left_Ankle-Left_Foot
- removed joint Biped__Left_Foot-Left_Toe
- removed joint Biped__Left_Hip-Top_Left_Leg
- removed joint Biped__Right_Ankle-Right_Foot
- removed joint Biped__Right_Foot-Right_Toe
- removed joint Biped__Right_Hip-Top_Right_Leg
- removed joint Biped__Top_Left_Leg-Bottom_Left_Leg
- removed joint Biped__Top_Right_Leg-Bottom_Right_Leg
- added joint l_ankle_flex: type revolute, parent Biped__Bottom_Left_Leg, child Biped__Left_Ankle, origin xyz=-1.50000000e-04  -2.21290000e-01  -1.13000000e-03 rpy=0  0  0, axis -1  0  0, limit lower=-1.36043531266 upper=0.135930877095 effort=100.0 velocity=0.0
- added joint l_ankle_roll: type revolute, parent Biped__Left_Ankle, child l_foot, origin xyz=-0.00077 -0.0179  -0.06914 rpy=0  0  0, axis 0      -0.00511  0.99998, limit lower=-1.32128191897 upper=1.32128191897 effort=100.0 velocity=0.0
- added joint l_hip_abduct: type revolute, parent pelvis, child Biped__Left_Hip, origin xyz=0.00302  0.05556  0.51514 rpy=1.56567  0      -1.57079, axis 0      -0.00511  0.99998, limit lower=-0.486936705914 upper=0.628150227902 effort=100.0 velocity=0.0
- added joint l_hip_flex: type revolute, parent Biped__Left_Hip, child Biped__Top_Left_Leg, origin xyz=-8.05900000e-02  -1.00000000e-05   3.02000000e-03 rpy=0  0  0, axis -1  0  0, limit lower=-2.03583339041 upper=2.16044300072 effort=100.0 velocity=0.0
- added joint l_knee: type revolute, parent Biped__Top_Left_Leg, child Biped__Bottom_Left_Leg, origin xyz=0.00373 -0.20954 -0.00107 rpy=0  0  0, axis -1  0  0, limit lower=-2.61562604133 upper=2.60767984583 effort=100.0 velocity=0.0
- added joint l_toe_flex: type revolute, parent l_foot, child l_toe, origin xyz=0.00232 -0.03426 -0.06708 rpy=0  0  0, axis -1  0  0, limit lower=-0.421908321567 upper=1.92797301525 effort=100.0 velocity=0.0
- added joint r_ankle_flex: type revolute, parent Biped__Bottom_Right_Leg, child Biped__Right_Ankle, origin xyz=4.00000000e-05  -2.21290000e-01  -1.13000000e-03 rpy=0  0  0, axis -1  0  0, limit lower=-1.34264425814 upper=0.135930877095 effort=100.0 velocity=0.0
- added joint r_ankle_roll: type revolute, parent Biped__Right_Ankle, child r_foot, origin xyz=-0.00079 -0.01789 -0.07124 rpy=0  0  0, axis 0       0.00511 -0.99998, limit lower=-1.32128191897 upper=1.32128191897 effort=100.0 velocity=0.0
- added joint r_hip_abduct: type revolute, parent pelvis, child Biped__Right_Hip, origin xyz=-0.00313 -0.05556  0.51514 rpy=1.56567  0      -1.57079, axis 0       0.00511 -0.99998, limit lower=-0.450917249297 upper=0.628150227902 effort=100.0 velocity=0.0
- added joint r_hip_flex: type revolute, parent Biped__Right_Hip, child Biped__Top_Right_Leg, origin xyz=7.52400000e-02   1.00000000e-05  -3.13000000e-03 rpy=0  0  0, axis -1  0  0, limit lower=-2.03583339041 upper=2.16044300072 effort=100.0 velocity=0.0
- added joint r_knee: type revolute, parent Biped__Top_Right_Leg, child Biped__Bottom_Right_Leg, origin xyz=0.00328 -0.20954 -0.00107 rpy=0  0  0, axis -1  0  0, limit lower=-2.60767984583 upper=2.60767984583 effort=100.0 velocity=0.0
- added joint r_toe_flex: type revolute, parent r_foot, child r_toe, origin xyz=0.00258 -0.03427 -0.06497 rpy=0  0  0, axis -1  0  0, limit lower=-0.421908321567 upper=1.92797301525 effort=100.0 velocity=0.0

Commit message: fix right toe contact points; add basic trajectory planner (currently attempts to go to a static pose); implement PD controller without using pdcontrol function (for extensibility); ignore all contact groups in controller except those on feet (heel/midfoot/toe) for better simulation performance.

File: urdf/Legs.urdf (robot description, URDF)
Before this commit: robot Legs, 13 links, 12 joints
Links:
- link r_toe: geometry collision mesh filename=meshes/Right_Toe_col.STL scale=1 1 1; collision sphere radius=0.0

Commit message: moved pelvis coordinates to inertial center

File: urdf/Legs.urdf (robot description, URDF)
Before this commit: robot Legs, 13 links, 12 joints
Links:
- link pelvis: geometry collision mesh filename=meshes/Body_col.STL scale=1 1 1; visual mesh filename=meshes/Body.obj scale=1 1 1
Joints:
- joint l_hip_abduct: origin xyz=0.00302  0.05556  0.51514 rpy=1.56567  0      -1.57079 -> xyz=0.0107    0.05539   -0.10919 rpy=1.56567  0      -1.57079
- joint r_hip_abduct: origin xyz=-0.00313 -0.05556  0.51514 rpy=1.56567  0      -1.57079 -> xyz=0.00455  -0.05573  -0.10919 rpy=1.56567  0      -1.57079

Commit message: moved foot frames to align with pelvis and world frames

File: urdf/Legs.urdf (robot description, URDF)
Before this commit: robot Legs, 13 links, 12 joints
Links:
- link l_foot: geometry collision mesh filename=meshes/Left_Foot_col.STL scale=1 1 1; collision sphere radius=0.0
- link l_toe: geometry collision mesh filename=meshes/Left_Toe_col.STL scale=1 1 1; visual mesh filename=meshes/Left_Toe.STL scale=1 1 1
- link r_foot: geometry collision mesh filename=meshes/Right_Foot_col.STL scale=1 1 1; collision sphere radius=0.0
Joints:
- joint l_ankle_roll: axis 0      -0.00511  0.99998 -> -0.99998      0  -0.00511; origin xyz=-0.00077 -0.0179  -0.06914 rpy=0  0  0 -> xyz=-0.00077 -0.0179  -0.06914 rpy=-1.5708  1.5708 0
- joint l_toe_flex: origin xyz=0.00232 -0.03426 -0.06708 rpy=0  0  0 -> xyz=0.06708 -0.00232 -0.03426 rpy=1.5708  0 -1.5708
- joint r_ankle_roll: axis 0       0.00511 -0.99998 -> 0.99998    0   0.00511; origin xyz=-0.00079 -0.01789 -0.07124 rpy=0  0  0 -> xyz=-0.00079 -0.01789 -0.07124 rpy=-1.5708  1.5708 0
- joint r_toe_flex: origin xyz=0.00258 -0.03427 -0.06497 rpy=0  0  0 -> xyz=0.06497 -0.00258 -0.03427 rpy=1.5708  0 -1.5708

Commit message: REMOVED TOES

File: urdf/Legs.urdf (robot description, URDF)
Before this commit: robot Legs, 13 links, 12 joints
Links:
- removed link l_toe
- removed link r_toe
Joints:
- removed joint l_toe_flex
- removed joint r_toe_flex
