Commit message: use actual extension in mesh paths

File: urdf/caminante_minimal.urdf (robot description, URDF)
Before this commit: robot caminante, 11 links, 10 joints
Links:
- link l_foot: geometry collision sphere radius=0.0; collision sphere radius=0.0
- link l_lglut: geometry visual mesh filename=meshes/Left_Hip.obj scale=1 1 1
- link l_lleg: geometry visual mesh filename=meshes/Bottom_Left_Leg.obj scale=1 1 1
- link l_talus: geometry visual mesh filename=meshes/Left_Ankle.obj scale=1 1 1
- link l_uleg: geometry visual mesh filename=meshes/Top_Left_Leg.obj scale=1 1 1
- link r_foot: geometry collision sphere radius=0.0; collision sphere radius=0.0
- link r_lglut: geometry visual mesh filename=meshes/Right_Hip.obj scale=1 1 1
- link r_lleg: geometry visual mesh filename=meshes/Bottom_Right_Leg.obj scale=1 1 1
- link r_talus: geometry visual mesh filename=meshes/Right_Ankle.obj scale=1 1 1
- link r_uleg: geometry visual mesh filename=meshes/Top_Right_Leg.obj scale=1 1 1

Commit message: add battery weight to pelvis

File: urdf/caminante_minimal.urdf (robot description, URDF)
Before this commit: robot caminante, 11 links, 10 joints
Links:
- link pelvis: mass 3.53324885586669 -> 6.4909068

Commit message: add 90 deg knee joint limit

File: urdf/caminante_minimal.urdf (robot description, URDF)
Before this commit: robot caminante, 11 links, 10 joints
Joints:
- joint l_leg_kny: limit lower=0 upper=2.35637 effort=890 velocity=12 -> lower=0 upper=1.57 effort=890 velocity=12
- joint r_leg_kny: limit lower=0 upper=2.35637 effort=890 velocity=12 -> lower=0 upper=1.57 effort=890 velocity=12
